Commit message: moveit2 setup

File: install/cobot_description/share/cobot_description/urdf/cobot_camera.urdf.xacro (robot description, xacro)
@@ -5,4 +5,5 @@
     <xacro:include filename="/home/fra/ros2_master_ws/src/cobot_description/urdf/custom_cobot_gazebo.xacro"/>
     <xacro:include filename="/home/fra/ros2_master_ws/src/cobot_description/urdf/camera.xacro"/>
+    <xacro:property name="gazebo_control" value="false" />
     <link name="world">
     </link>
@@ -71,85 +72,87 @@
     </joint>
     <xacro:custom_gripper parent="tool0" origin_xyz="0 0 0" />
-    <ros2_control name="GazeboSystem" type="system">
-        <hardware>
-            <plugin>gazebo_ros2_control/GazeboSystem</plugin>
-        </hardware>
-        <joint name="base_link__link1">
-            <command_interface name="position">
-                <param name="min">-6.28</param>
-                <param name="max">6.28</param>
-            </command_interface>
-            <state_interface name="position">
-                <param name="initial_value">0.0</param>
-            </state_interface>
-            <state_interface name="velocity" />
-        </joint>
-        <joint name="link1__link2">
-            <command_interface name="position">
-                <param name="min">-6.28</param>
-                <param name="max">6.28</param>
-            </command_interface>
-            <state_interface name="position" >
-                <param name="initial_value">0.0</param>
-            </state_interface>
-            <state_interface name="velocity" />
-        </joint>
-        <joint name="link2__link3">
-            <command_interface name="position">
-                <param name="min">-6.28</param>
-                <param name="max">6.28</param>
-            </command_interface>
-            <state_interface name="position" >
-                <param name="initial_value">0.0</param>
-            </state_interface>
-            <state_interface name="velocity" />
-        </joint>
-        <joint name="link3__link4">
-            <command_interface name="position">
-                <param name="min">-6.28</param>
-                <param name="max">6.28</param>
-            </command_interface>
-            <state_interface name="position" >
-                <param name="initial_value">0.0</param>
-            </state_interface>
-            <state_interface name="velocity" />
-        </joint>
-        <joint name="link4__link5">
-            <command_interface name="position">
-                <param name="min">-6.28</param>
-                <param name="max">6.28</param>
-            </command_interface>
-            <state_interface name="position" >
-                <param name="initial_value">0.0</param>
-            </state_interface>
-            <state_interface name="velocity" />
-        </joint>
-        <joint name="link5__link6">
-            <command_interface name="position">
-                <param name="min">-6.28</param>
-                <param name="max">6.28</param>
-            </command_interface>
-            <state_interface name="position" >
-                <param name="initial_value">0.0</param>
-            </state_interface>
-            <state_interface name="velocity" />
-        </joint>
-        <joint name="finger_right_joint">
-            <command_interface name="position" />
-            <state_interface name="position" >
-                <param name="initial_value">0.0</param>
-            </state_interface>
-            <state_interface name="velocity" />
-        </joint>
-        <joint name="finger_left_joint">
-            <param name="mimic">finger_right_joint</param>
-            <param name="multiplier">-1</param>
-            <command_interface name="position" />
-            <state_interface name="position" >
-                <param name="initial_value">0.0</param>
-            </state_interface>
-            <state_interface name="velocity" />
-        </joint>
-    </ros2_control>
+    <xacro:if value="${gazebo_control}">
+        <ros2_control name="GazeboSystem" type="system">
+            <hardware>
+                <plugin>gazebo_ros2_control/GazeboSystem</plugin>
+            </hardware>
+            <joint name="base_link__link1">
+                <command_interface name="position">
+                    <param name="min">-6.28</param>
+                    <param name="max">6.28</param>
+                </command_interface>
+                <state_interface name="position">
+                    <param name="initial_value">0.0</param>
+                </state_interface>
+                <state_interface name="velocity" />
+            </joint>
+            <joint name="link1__link2">
+                <command_interface name="position">
+                    <param name="min">-6.28</param>
+                    <param name="max">6.28</param>
+                </command_interface>
+                <state_interface name="position" >
+                    <param name="initial_value">0.0</param>
+                </state_interface>
+                <state_interface name="velocity" />
+            </joint>
+            <joint name="link2__link3">
+                <command_interface name="position">
+                    <param name="min">-6.28</param>
+                    <param name="max">6.28</param>
+                </command_interface>
+                <state_interface name="position" >
+                    <param name="initial_value">0.0</param>
+                </state_interface>
+                <state_interface name="velocity" />
+            </joint>
+            <joint name="link3__link4">
+                <command_interface name="position">
+                    <param name="min">-6.28</param>
+                    <param name="max">6.28</param>
+                </command_interface>
+                <state_interface name="position" >
+                    <param name="initial_value">0.0</param>
+                </state_interface>
+                <state_interface name="velocity" />
+            </joint>
+            <joint name="link4__link5">
+                <command_interface name="position">
+                    <param name="min">-6.28</param>
+                    <param name="max">6.28</param>
+                </command_interface>
+                <state_interface name="position" >
+                    <param name="initial_value">0.0</param>
+                </state_interface>
+                <state_interface name="velocity" />
+            </joint>
+            <joint name="link5__link6">
+                <command_interface name="position">
+                    <param name="min">-6.28</param>
+                    <param name="max">6.28</param>
+                </command_interface>
+                <state_interface name="position" >
+                    <param name="initial_value">0.0</param>
+                </state_interface>
+                <state_interface name="velocity" />
+            </joint>
+            <joint name="finger_right_joint">
+                <command_interface name="position" />
+                <state_interface name="position" >
+                    <param name="initial_value">0.0</param>
+                </state_interface>
+                <state_interface name="velocity" />
+            </joint>
+            <joint name="finger_left_joint">
+                <param name="mimic">finger_right_joint</param>
+                <param name="multiplier">-1</param>
+                <command_interface name="position" />
+                <state_interface name="position" >
+                    <param name="initial_value">0.0</param>
+                </state_interface>
+                <state_interface name="velocity" />
+            </joint>
+        </ros2_control>
+    </xacro:if>
     <gazebo>
         <plugin filename="libgazebo_ros2_control.so" name="gazebo_ros2_control">
