Commit message: moveit gazebo interface

File: install/custom_robot_moveit_config/share/custom_robot_moveit_config/config/custom_robot.ros2_control.xacro (robot description, xacro)
@@ -6,5 +6,6 @@
             <hardware>
                 <!-- By default, set up controllers for simulation. This won't work on real hardware -->
-                <plugin>mock_components/GenericSystem</plugin>
+                <!-- <plugin>mock_components/GenericSystem</plugin> -->
+                <plugin>gazebo_ros2_control/GazeboSystem</plugin>
             </hardware>
             <joint name="base_link__link1">
@@ -57,4 +58,13 @@
                 <state_interface name="velocity"/>
             </joint>
+            <joint name="finger_left_joint">
+                <param name="mimic">finger_right_joint</param>
+                <param name="multiplier">-1</param>
+                <command_interface name="position" />
+                <state_interface name="position" >
+                    <param name="initial_value">0.0</param>
+                </state_interface>
+                <state_interface name="velocity" />
+            </joint>
         </ros2_control>
     </xacro:macro>
